File: Hardware/GomuGomuNoDrive_hard/Rubber_drive_hard.kicad_sch (KiCad schematic)
At the start: 67 parts, among them J1 9V, J2 AudioJack3, J3 AudioJack3, J4 Conn_02x03_Counter_Clockwise, Q10 BC550, Q4 TN2106, Q5 TN2106, Q9 BC550, SW1 SW_DPDT_x2, SW10 SW_DPDT_x2, SW11 SW_SPDT, SW2 SW_DPDT_x2, SW3 SW_DPDT_x2, SW4 SW_DPDT_x2, SW5 SW_SPDT_MSM, SW6 SW_SPDT_MSM, SW7 SW_DPDT_x2, SW8 SW_DPDT_x2, U2 TC7662Bx0A, U5 OPA1679

Commit message: Correct Schematic/PCB for Hard clip pedal
Parts:
- removed C4: 47u, Capacitor_SMD:CP_Elec_6.3x5.4, symbol Brutalizer Jr-rescue:CP1-Device
- removed J4: Conn_02x03_Counter_Clockwise, Connector_PinHeader_2.54mm:PinHeader_2x03_P2.54mm_Vertical, symbol Connector_Generic:Conn_02x03_Counter_Clockwise
- removed Q10, Q9: BC550, Package_TO_SOT_THT:TO-92_Wide, symbol Transistor_BJT:Q_NPN_CBE
- removed Q4, Q5: TN2106, Package_TO_SOT_THT:TO-92_Inline, symbol Transistor_FET:BS170
- removed R7: 10K, Resistor_SMD:R_1206_3216Metric_Pad1.30x1.75mm_HandSolder, symbol Device:R
- removed SW1, SW2: SW_DPDT_x2, Button_Switch_THT:SW_CK_JS202011CQN_DPDT_Straight, symbol Switch:SW_DPDT_x2
- removed unit 2 of SW3
- removed unit 2 of SW4
- removed TP26: out, Connector_PinHeader_2.54mm:PinHeader_1x01_P2.54mm_Vertical, symbol Connector:TestPoint
- added C18: 10u, Capacitor_SMD:C_0805_2012Metric_Pad1.18x1.45mm_HandSolder, symbol Device:C
- added J5: Conn_01x06_Socket, Connector_JST:JST_EH_B6B-EH-A_1x06_P2.50mm_Vertical, symbol Connector:Conn_01x06_Socket
- added Q1, Q2: BC850, Package_TO_SOT_SMD:SOT-23, symbol Transistor_BJT:BC850
- C1, C10, C11, C12, C13, C14, C15, C16, C17, C2, C5, C8, C9: footprint Capacitor_SMD:C_1206_3216Metric_Pad1.33x1.80mm_HandSolder -> Capacitor_SMD:C_0805_2012Metric_Pad1.18x1.45mm_HandSolder
- C3: value 10n -> 4n7; footprint Capacitor_SMD:C_1206_3216Metric_Pad1.33x1.80mm_HandSolder -> Capacitor_SMD:C_0805_2012Metric_Pad1.18x1.45mm_HandSolder
- C6: value C -> 220n; footprint Capacitor_SMD:C_1206_3216Metric_Pad1.33x1.80mm_HandSolder -> Capacitor_SMD:C_0805_2012Metric_Pad1.18x1.45mm_HandSolder
- C7: value 10n -> 22n; footprint Capacitor_SMD:C_1206_3216Metric_Pad1.33x1.80mm_HandSolder -> Capacitor_SMD:C_0805_2012Metric_Pad1.18x1.45mm_HandSolder
- D1: value BAT42W -> C8598
- D2: value BAT41 -> C8598
- D3: value 1N5818 -> C8598
- R10, R11, R13, R16, R17: footprint Resistor_SMD:R_1206_3216Metric_Pad1.30x1.75mm_HandSolder -> Resistor_SMD:R_0805_2012Metric_Pad1.20x1.40mm_HandSolder
- R12, R14: value 4K7 -> 100; footprint Resistor_SMD:R_1206_3216Metric_Pad1.30x1.75mm_HandSolder -> Resistor_SMD:R_0805_2012Metric_Pad1.20x1.40mm_HandSolder
- R15: value 1M -> 100; footprint Resistor_SMD:R_1206_3216Metric_Pad1.30x1.75mm_HandSolder -> Resistor_SMD:R_0805_2012Metric_Pad1.20x1.40mm_HandSolder
- R9: value R -> 6K8; footprint Resistor_SMD:R_1206_3216Metric_Pad1.30x1.75mm_HandSolder -> Resistor_SMD:R_0805_2012Metric_Pad1.20x1.40mm_HandSolder
- RV11: value R_Potentiometer -> 100K_Log
- RV12, RV5, RV6, RV8: value 100? -> 5K
- RV21: value 1M -> 100K Log
- TP25: value post_diode_DC -> GND
Connections:
- net 9V: now also U2.8 (V+), C18.2
- net CircuitInput: now also J5.5 (Pin_5)
- net GND: now also J1.1, RV21.1, TP25.1, C18.1, J5.1 (Pin_1), Q2.2 (E); no longer J1.2, R15.1
- net JackInput_tip: now also J5.3 (Pin_3)
- net JackOutput_tip: now also J5.6 (Pin_6)
- net LED_CATHODE: now also J5.2 (Pin_2)
- net Rubber_hard_north: now also Q1.2 (E)
- net V: now also J1.2; no longer J1.1
- net out: now also R15.2, J5.4 (Pin_4); no longer RV21.2, U5.8
- net at C3.2, C7.2, RV4.2: now also Q1.1 (B)
- net at TP24.1, U5.6 (-), U5.7: now also C6.1
- net at C2.2, C5.2, RV3.2: now also Q2.1 (B)
- net at C9.1, RV8.2: now also Q1.3 (C)
- net at C17.2, RV5.2: now also Q2.3 (C)
- net at U5.12 (+): now also RV21.2
- net at U5.13 (-): now also R15.1, U5.14
- new net: C6.2, RV21.3
- new net: U5.8, U5.9 (-)
- no-connect marks 22 -> 12
Other:
- note added: "ROGNER un peu pour rentrer dans boitier"
- note added: "input vol hard 100m/300mvV -> a few V"
- note removed: "input vol hard 100mV -> a few V"
- moved on the sheet: C10, C14, C15, D3, J1, TP24, TP27, U5B, U5D, U5E
